File: Audiophi Hat+.kicad_sch (KiCad schematic)
At the start: 31 parts, among them IC2 CAT24C32WI-GT3JN, IC3 AP3441SHE-7B, J1 PINHD_1x2_Male, J2 936, J3 936, U1 PEC11H-4015F-S0016

Commit message: Update
Parts:
- added C1: 1nF_0603_50V, Capacitor_SMD:C_0603_1608Metric, symbol PCM_4ms_Capacitor:1nF_0603_50V
- added C15, C3: 0.1uF, 16V, SamacSys_Parts:CAPC1608X90N, symbol SamacSys_Parts:GCM188R71C104JA37D
- added FL1: BLM18AG102BH1D, SamacSys_Parts:BLM18AG102BH1D, symbol SamacSys_Parts:BLM18AG102BH1D
- added J4: RCA FEMALE, 936, symbol SamacSys_Parts:936
- added R1: 22R, SamacSys_Parts:RESC1608X55N, symbol SamacSys_Parts:RC0603JR-0722RL
- added R2: 75R_0603, PCM_Resistor_SMD_AKL:R_0603_1608Metric, symbol PCM_4ms_Resistor:75R_0603
- added RN1: 22R, symbol Device:R_Pack04
- added U2: WM8960CGEFL_V, SamacSys_Parts:QFN50P500X500X100-33N, symbol SamacSys_Parts:WM8960CGEFL_V
- added Y1: ISM97-3251BH-24.000MHz, SamacSys_Parts:ISM973251BH24000MHz, symbol SamacSys_Parts:ISM97-3251BH-24.000MHz
Connections:
- net +3.3V: now also FL1.1
- net GND: now also C1.1, C3.1, J4.MH1, J4.MH2, J4.MH3, R2.2, Y1.2 (CASE/GROUND)
- new net: C15.1, J4.1, R2.1
- new net: R1.1, Y1.3 (OUTPUT)
- new net: C1.2, C3.2, FL1.2, Y1.4 (SUPPLY_VOLTAGE)
- new net MCLK: R1.2
- no-connect marks 4 -> 5
Other:
- note added: "CRYSTAL 24MHZ MCLK INPUT"
- company: (none) -> Audiophi
- title: (none) -> Audiophi Hat+
- moved on the sheet: C10, C11, C12, C13, C14, C2, C4, C5, C6, C7, C8, C9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
